Commit message: add joint_state_publisher_node to launch

File: diff_bot/urdf/properties.xacro (robot description, xacro)
@@ -8,15 +8,15 @@
     <xacro:property name="chassis_mass" value="3.0"/>
     <!-- Wheels -->
-    <xacro:property name="wheel_offset_x" value="0.1"/>
-    <xacro:property name="wheel_offset_y" value="0.41"/>
+    <xacro:property name="wheel_offset_x" value="0.16"/>
+    <xacro:property name="wheel_offset_y" value="0.226"/>
     <xacro:property name="wheel_offset_z" value="-0.025"/>
-    <xacro:property name="wheel_thickness" value="0.03"/>
+    <xacro:property name="wheel_thickness" value="0.05"/>
     <xacro:property name="wheel_radius" value="0.08"/>
     <xacro:property name="wheel_mass" value="0.04"/>
     <!-- Caster Wheel -->
-    <xacro:property name="caster_wheel_radius" value="0.01"/>
+    <xacro:property name="caster_wheel_radius" value="0.055"/>
     <xacro:property name="caster_wheel_mass" value="0.01"/>
     <xacro:property name="caster_wheel_offset_x" value="0.6"/>
-    <xacro:property name="caster_wheel_offset_z" value="-0.035"/>
+    <xacro:property name="caster_wheel_offset_z" value="-0.05"/>
     <!-- Colors -->
     <material name="white">

File: diff_bot/urdf/robot.urdf.xacro (robot description, xacro)
@@ -4,4 +4,6 @@
   <xacro:include filename="inertial_macros.xacro"/>
   <xacro:include filename="chassis.xacro"/>
+  <xacro:include filename="wheels.xacro"/>
+  <xacro:include filename="caster_wheel.xacro"/>
   <!-- Base Link -->
   <link name="base_link"/>
