Commit message: ..

File: diff_bot/urdf/chassis.xacro (robot description, xacro)
@@ -1,5 +1,5 @@
 <?xml version="1.0"?>
 <robot xmlns:xacro="http://www.ros.org/wiki/xacro">
-        <!-- Chassis Link -->
+    <!-- Chassis Link -->
     <link name="chassis_link">
         <visual>
@@ -11,9 +11,9 @@
         </visual>
         <collision>
+            <geometry>
+                <box size="${chassis_length} ${chassis_width} ${chassis_height}"/>
+            </geometry>
             <origin xyz="${chassis_length/2} 0.0 ${chassis_height/2}"/>
         </collision>
-        <xacro:inertial_box mass="${chassis_mass}" x="${chassis_length}" y="${chassis_width}" z="${chassis_height}">
-            <origin xyz="${chassis_length/2} 0 ${chassis_height/2}" rpy="0 0 0"/>
-        </xacro:inertial_box>
     </link>
     <!-- Chassis joint -->

File: diff_bot/urdf/wheels.xacro (robot description, xacro)
@@ -1,45 +1,46 @@
 <?xml version="1.0"?>
 <robot xmlns:xacro="http://www.ros.org/wiki/xacro">
-    <!-- Wheel Link Macro -->
-    <xacro:macro name="wheel_link" params="link_name">
-        <link name="${link_name}">
-            <visual>
-                <geometry>
-                    <cylinder radius="${wheel_radius}" length="${wheel_thickness}"/>
-                </geometry>
-                <material name="red"/>
-            </visual>
-            <collision>
-                <geometry>
-                    <sphere radius="${wheel_radius}"/>
-                </geometry>
-            </collision>
-            <xacro:inertial_cylinder mass="${wheel_mass}" length="${wheel_thickness}" radius="${wheel_radius}">
-            <origin xyz="0 0 0" rpy="0 0 0"/>
-        </xacro:inertial_cylinder>
-        </link>
-    </xacro:macro>
-    <!-- Wheel Joint Macro -->
-    <xacro:macro name="wheel_joint" params="joint_name wheel_name y_offset ">
-        <joint name="${joint_name}" type="continuous">
-            <origin xyz="${wheel_offset_x} ${y_offset} ${wheel_offset_z}" rpy="${-pi/2} 0.0 0.0"/>
-            <parent link="base_link"/>
-            <child link="${wheel_name}"/>
-            <axis xyz="0.0 0.0 1"/>
-        </joint>
-    </xacro:macro>
-    <!-- Left Wheel Link -->
-    <xacro:wheel_link link_name="left_wheel_link" />
-    <!-- Left Wheel Joint -->
-    <xacro:wheel_joint joint_name="left_wheel_joint" wheel_name="left_wheel_link" y_offset="${wheel_offset_y}"/>
-    <!-- Right Wheel Link -->
-    <xacro:wheel_link link_name="right_wheel_link" />
-    <!-- Right Wheel Joint -->
-    <xacro:wheel_joint joint_name="right_wheel_joint" wheel_name="right_wheel_link" y_offset="${-wheel_offset_y}"/>
-    <gazebo reference="left_wheel_link">
-        <material> Gazebo/Black </material>
-    </gazebo>
-    <gazebo reference="right_wheel_link">
-        <material> Gazebo/Black </material>
-    </gazebo>
+  <!-- Wheel Link Macro -->
+  <xacro:macro name="wheel_link" params="link_name">
+    <link name="${link_name}">
+      <visual>
+        <origin xyz="0 0 0" rpy="0 0 0"/>
+        <geometry>
+          <cylinder radius="${wheel_radius}" length="${wheel_thickness}"/>
+        </geometry>
+        <material name="red"/>
+      </visual>
+      <collision>
+        <origin xyz="0 0 0" rpy="0 0 0"/>
+        <geometry>
+          <cylinder radius="${wheel_radius}" length="${wheel_thickness}"/>
+        </geometry>
+      </collision>
+      <xacro:inertial_cylinder mass="${wheel_mass}" length="${wheel_thickness}" radius="${wheel_radius}">
+        <origin xyz="0 0 0" rpy="0 0 0"/>
+      </xacro:inertial_cylinder>
+    </link>
+  </xacro:macro>
+  <!-- Wheel Joint Macro -->
+  <xacro:macro name="wheel_joint" params="joint_name wheel_name y_offset">
+    <joint name="${joint_name}" type="continuous">
+      <origin xyz="${wheel_offset_x} ${y_offset} ${wheel_offset_z}" rpy="${-pi/2} 0 0"/>
+      <parent link="base_link"/>
+      <child link="${wheel_name}"/>
+      <axis xyz="0 0 1"/>
+    </joint>
+  </xacro:macro>
+  <!-- Left Wheel -->
+  <xacro:wheel_link link_name="left_wheel_link"/>
+  <xacro:wheel_joint joint_name="left_wheel_joint" wheel_name="left_wheel_link" y_offset="${wheel_offset_y}"/>
+  <!-- Right Wheel -->
+  <xacro:wheel_link link_name="right_wheel_link"/>
+  <xacro:wheel_joint joint_name="right_wheel_joint" wheel_name="right_wheel_link" y_offset="${-wheel_offset_y}"/>
+  <!-- Gazebo Materials -->
+  <gazebo reference="left_wheel_link">
+    <material>Gazebo/Black</material>
+  </gazebo>
+  <gazebo reference="right_wheel_link">
+    <material>Gazebo/Black</material>
+  </gazebo>
 </robot>
